Commit message: Init

File: living_lab_robot_description/urdf/arm.urdf.xacro (robot description, xacro)
@@ -15,7 +15,7 @@
         </collision>
         <inertial>
-            <origin xyz="0 0 0" rpy="0 0 0"/>
-            <mass value="1.0"/>
-            <inertia ixx="1.0" ixy="0.0" ixz="0.0" iyy="1.0" iyz="0.0" izz="1.0"/>
+            <origin xyz="0.0784 0 -0.0345" rpy="0 0 0"/>
+            <mass value="0.04997"/>
+            <inertia ixx="0.0007768" ixy="0.0" ixz="0.0" iyy="0.0023504" iyz="0.0" izz="0.0020179"/>
         </inertial>
     </link>
@@ -25,5 +25,6 @@
         <origin xyz="0.035 0 -0.0228" rpy="0 0 0"/>
         <axis xyz="1 0 0"/>
-        <limit lower="0" upper="0" velocity="1.0" effort="1000"/>
+        <limit lower="-0.15" upper="0" velocity="0.06" effort="50"/>
+        <dynamics damping="0.01" friction="0.0"/>
     </joint>
     <xacro:insert_position_transmission name="arm_base_joint" />
@@ -42,7 +43,7 @@
         </collision>
         <inertial>
-            <origin xyz="0 0 0" rpy="0 0 0"/>
-            <mass value="1.0"/>
-            <inertia ixx="1.0" ixy="0.0" ixz="0.0" iyy="1.0" iyz="0.0" izz="1.0"/>
+            <origin xyz="0.0330 0 0" rpy="0 0 0"/>
+            <mass value="0.05067"/>
+            <inertia ixx="0.0021992" ixy="0.0" ixz="0.0" iyy="0.0006670" iyz="0.0" izz="0.0021992"/>
         </inertial>
     </link>
@@ -52,5 +53,6 @@
         <origin xyz="0.15612 0 -0.051215" rpy="0 0 0"/>
         <axis xyz="1 0 0"/>
-        <limit lower="${-180/180*pi}" upper="${180/180*pi}" velocity="0.4" effort="1000"/>
+        <limit lower="${-180/180*pi}" upper="${180/180*pi}" velocity="1.0" effort="50"/>
+        <dynamics damping="0.01" friction="0.0"/>
     </joint>
     <xacro:insert_position_transmission name="arm1_joint" />
@@ -69,7 +71,7 @@
         </collision>
         <inertial>
-            <origin xyz="0 0 0" rpy="0 0 0"/>
-            <mass value="1.0"/>
-            <inertia ixx="1.0" ixy="0.0" ixz="0.0" iyy="1.0" iyz="0.0" izz="1.0"/>
+            <origin xyz="0.1642 0 0.0083" rpy="0 0 0"/>
+            <mass value="0.09000"/>
+            <inertia ixx="0.0021659" ixy="0" ixz="0" iyy="0.0074914" iyz="0" izz="0.0086634"/>
         </inertial>
     </link>
@@ -79,5 +81,6 @@
         <origin xyz="0.033 0 0" rpy="0 0 0"/>
         <axis xyz="0 1 0"/>
-        <limit lower="${-95/180*pi}" upper="${95/180*pi}" velocity="0.4" effort="1000"/>
+        <limit lower="${-95/180*pi}" upper="${95/180*pi}" velocity="1.0" effort="50"/>
+        <dynamics damping="0.01" friction="0.0"/>
     </joint>
     <xacro:insert_position_transmission name="arm2_joint" />
@@ -96,7 +99,7 @@
         </collision>
         <inertial>
-            <origin xyz="0 0 0" rpy="0 0 0"/>
-            <mass value="1.0"/>
-            <inertia ixx="1.0" ixy="0.0" ixz="0.0" iyy="1.0" iyz="0.0" izz="1.0"/>
+            <origin xyz="0.1137 0 -0.0409" rpy="0 0 0"/>
+            <mass value="0.08000"/>
+            <inertia ixx="0.0013151" ixy="0" ixz="0" iyy="0.0034294" iyz="0.0" izz="0.0042325"/>
         </inertial>
     </link>
@@ -106,5 +109,6 @@
         <origin xyz="0.264 0 0.030" rpy="0 0 0"/>
         <axis xyz="0 1 0"/>
-        <limit lower="${-180/180*pi}" upper="${5/180*pi}" velocity="0.4" effort="1000"/>
+        <limit lower="${-180/180*pi}" upper="${5/180*pi}" velocity="1.0" effort="50"/>
+        <dynamics damping="0.01" friction="0.0"/>
     </joint>
     <xacro:insert_position_transmission name="arm3_joint" />
@@ -123,7 +127,7 @@
         </collision>
         <inertial>
-            <origin xyz="0 0 0" rpy="0 0 0"/>
-            <mass value="1.0"/>
-            <inertia ixx="1.0" ixy="0.0" ixz="0.0" iyy="1.0" iyz="0.0" izz="1.0"/>
+            <origin xyz="0.0269 0.0 0.0" rpy="0 0 0"/>
+            <mass value="0.02697"/>
+            <inertia ixx="00.0012527" ixy="0.0" ixz="0.0" iyy="0.0003956" iyz="0.0" izz="0.0012527"/>
         </inertial>
     </link>
@@ -133,5 +137,6 @@
         <origin xyz="0.231 0 -0.042" rpy="0 0 0"/>
         <axis xyz="1 0 0"/>
-        <limit lower="${-180/180*pi}" upper="${180/180*pi}" velocity="0.4" effort="1000"/>
+        <limit lower="${-180/180*pi}" upper="${180/180*pi}" velocity="1.0" effort="50"/>
+        <dynamics damping="0.01" friction="0.0"/>
     </joint>
     <xacro:insert_position_transmission name="arm4_joint" />
@@ -150,7 +155,7 @@
         </collision>
         <inertial>
-            <origin xyz="0 0 0" rpy="0 0 0"/>
-            <mass value="1.0"/>
-            <inertia ixx="1.0" ixy="0.0" ixz="0.0" iyy="1.0" iyz="0.0" izz="1.0"/>
+            <origin xyz="0.0667 0 -0.0005" rpy="0 0 0"/>
+            <mass value="0.03885"/>
+            <inertia ixx="0.0005947" ixy="0.0" ixz="0.0" iyy="0.0005919" iyz="0.0" izz="0.0010050"/>
         </inertial>
     </link>
@@ -160,12 +165,25 @@
         <origin xyz="0.027 0 0" rpy="0 0 0"/>
         <axis xyz="0 1 0"/>
-        <limit lower="${-95/180*pi}" upper="${95/180*pi}" velocity="0.4" effort="1000"/>
+        <limit lower="${-95/180*pi}" upper="${95/180*pi}" velocity="1.0" effort="50"/>
+        <dynamics damping="0.01" friction="0.0"/>
     </joint>
     <xacro:insert_position_transmission name="arm5_joint" />
     <link name="arm_link6">
+        <visual>
+            <origin xyz="0 0 0" rpy="0 0 0"/>
+            <geometry>
+                <mesh filename="package://living_lab_robot_description/meshes/arm_link6.dae" scale="1 1 1"/>
+            </geometry>
+        </visual>
+        <collision>
+            <origin xyz="0 0 0" rpy="0 0 0"/>
+            <geometry>
+                <mesh filename="package://living_lab_robot_description/meshes/arm_link6.dae" scale="1 1 1"/>
+            </geometry>
+        </collision>
         <inertial>
-            <origin xyz="0 0 0" rpy="0 0 0"/>
-            <mass value="1.0"/>
-            <inertia ixx="1.0" ixy="0.0" ixz="0.0" iyy="1.0" iyz="0.0" izz="1.0"/>
+            <origin xyz="-0.0030 0 0" rpy="0 0 0"/>
+            <mass value="0.0038"/>
+            <inertia ixx="0.0000301" ixy="0.0" ixz="0.0" iyy="0.0000156" iyz="0.0" izz="0.0000156"/>
         </inertial>
     </link>
@@ -175,5 +193,6 @@
         <origin xyz="0.123 0 0" rpy="0 0 0"/>
         <axis xyz="1 0 0"/>
-        <limit lower="${-180/180*pi}" upper="${180/180*pi}" velocity="0.4" effort="1000"/>
+        <limit lower="${-180/180*pi}" upper="${180/180*pi}" velocity="1.0" effort="50"/>
+        <dynamics damping="0.01" friction="0.0"/>
     </joint>
     <xacro:insert_position_transmission name="arm6_joint" />

File: living_lab_robot_description/urdf/body_assy.urdf.xacro (robot description, xacro)
@@ -15,7 +15,7 @@
         </collision>
         <inertial>
-            <origin xyz="0 0 0" rpy="0 0 0"/>
-            <mass value="5.0"/>
-            <inertia ixx="1.0" ixy="0.0" ixz="0.0" iyy="1.0" iyz="0.0" izz="1.0"/>
+            <origin xyz="0 0 0.3780" rpy="0 0 0"/>
+            <mass value="30.21"/>
+            <inertia ixx="0.263797" ixy="0.000014" ixz="-0.000365" iyy="0.255334" iyz="-0.000303" izz="0.069846"/>
         </inertial>
     </link>
@@ -25,5 +25,5 @@
         <origin xyz="0 0 0.242" rpy="0 0 0"/>
         <axis xyz="0 0 1"/>
-        <limit lower="${-200/180*pi}" upper="${200/180*pi}" velocity="1.0" effort="1000"/>
+        <limit lower="${-200/180*pi}" upper="${200/180*pi}" velocity="0.4" effort="1000"/>
     </joint>
     <xacro:insert_position_transmission name="body_rotate_joint" />
@@ -43,6 +43,6 @@
         <inertial>
             <origin xyz="0 0 0" rpy="0 0 0"/>
-            <mass value="1.0"/>
-            <inertia ixx="1.0" ixy="0.0" ixz="0.0" iyy="1.0" iyz="0.0" izz="1.0"/>
+            <mass value="10.31"/>
+            <inertia ixx="0.001422" ixy="0" ixz="0" iyy="0.000917" iyz="0" izz="0.001769"/>
         </inertial>
     </link>
@@ -52,5 +52,6 @@
         <origin xyz="-0.05 0 0.665" rpy="0 0 0"/>
         <axis xyz="0 0 1"/>
-        <limit lower="-0.45" upper="0" velocity="0.04" effort="1000"/>
+        <limit lower="-0.45" upper="0" velocity="0.1" effort="100"/>
+        <dynamics damping="0.01" friction="0.0"/>
     </joint>
     <xacro:insert_position_transmission name="elevation_joint" />

File: living_lab_robot_description/urdf/gazebo.urdf.xacro (robot description, xacro)
@@ -12,8 +12,33 @@
             <odometryTopic>odom</odometryTopic>
             <odometryFrame>odom</odometryFrame>
-            <odometryRate>30.0</odometryRate>
+            <odometryRate>50.0</odometryRate>
             <robotBaseFrame>base_footprint</robotBaseFrame>
         </plugin>
     </gazebo>
+    <gazebo reference="omni_wheel_1">
+        <selfCollide>false</selfCollide>
+        <mu1 value="0.0"/>
+        <mu1 value="0.0"/>
+    </gazebo>
+    <gazebo reference="omni_wheel_2">
+        <selfCollide>false</selfCollide>
+        <mu1 value="0.0"/>
+        <mu1 value="0.0"/>
+    </gazebo>
+    <gazebo reference="omni_wheel_3">
+        <selfCollide>false</selfCollide>
+        <mu1 value="0.0"/>
+        <mu1 value="0.0"/>
+    </gazebo>
+    <xacro:macro name="insert_mimic_joint" params="reference name multiplier offset">
+        <gazebo>
+            <plugin name="mimic_${name}" filename="libgazebo_mimic_joint_plugin.so">
+                <joint>${reference}</joint>
+                <mimicJoint>${name}</mimicJoint>
+                <multiplier>${multiplier}</multiplier>
+                <offset>${offset}</offset>
+            </plugin>
+        </gazebo>
+    </xacro:macro>
     <gazebo reference="base_link">
         <mu1 value="0.0"/>
@@ -31,6 +56,6 @@
                             <samples>720</samples>
                             <resolution>1</resolution>
-                            <min_angle>-1.5707</min_angle>
-                            <max_angle>1.5707</max_angle>
+                            <min_angle>-1.5</min_angle>
+                            <max_angle>1.5</max_angle>
                         </horizontal>
                     </scan>

File: living_lab_robot_description/urdf/head_assy.urdf.xacro (robot description, xacro)
@@ -16,7 +16,7 @@
         </collision>
         <inertial>
-            <origin xyz="0 0 0" rpy="0 0 0"/>
-            <mass value="1.0"/>
-            <inertia ixx="1.0" ixy="0.0" ixz="0.0" iyy="1.0" iyz="0.0" izz="1.0"/>
+            <origin xyz="0 0 -0.1224" rpy="0 0 0"/>
+            <mass value="16.545411"/>
+            <inertia ixx="0.085366" ixy="0.0" ixz="0.0" iyy="0.085366" iyz="0.0" izz="0.105357"/>
         </inertial>
     </link>
@@ -43,7 +43,7 @@
         </collision>
         <inertial>
-            <origin xyz="0 0 0" rpy="0 0 0"/>
-            <mass value="1.0"/>
-            <inertia ixx="1.0" ixy="0.0" ixz="0.0" iyy="1.0" iyz="0.0" izz="1.0"/>
+            <origin xyz="0.014478 0.0 -0.045490" rpy="0 0 0"/>
+            <mass value="10.186690"/>
+            <inertia ixx="0.000811" ixy="0.0" ixz="0.000012" iyy="0.000271" iyz="0.0" izz="0.000576"/>
         </inertial>
     </link>
@@ -70,7 +70,7 @@
         </collision>
         <inertial>
-            <origin xyz="0 0 0" rpy="0 0 0"/>
-            <mass value="5.0"/>
-            <inertia ixx="1.0" ixy="0.0" ixz="0.0" iyy="1.0" iyz="0.0" izz="1.0"/>
+            <origin xyz="-0.098000 0 0.057616" rpy="0 0 0"/>
+            <mass value="20.540090"/>
+            <inertia ixx="0.022353" ixy="0.0" ixz="0.0" iyy="0.022353" iyz="0.0" izz="0.040886"/>
         </inertial>
     </link>
@@ -88,9 +88,9 @@
     <xacro:insert_rgbd_camera_sensor name="camera"/>
     <link name="gaze_link">
-        <inertial>
+        <!-- <inertial>
             <origin xyz="0 0 0" rpy="0 0 0"/>
-            <mass value="1.0"/>
-            <inertia ixx="1.0" ixy="0.0" ixz="0.0" iyy="1.0" iyz="0.0" izz="1.0"/>
-        </inertial>
+            <mass value="0.01"/>
+            <inertia ixx="0.0001" ixy="0.0" ixz="0.0" iyy="0.0001" iyz="0.0" izz="0.0001"/>
+        </inertial> -->
     </link>
     <joint name="gaze_fixed_joint" type="fixed">

File: living_lab_robot_description/urdf/mobile_assy.urdf.xacro (robot description, xacro)
@@ -16,7 +16,7 @@
         </collision>
         <inertial>
-            <origin xyz="0 0 0" rpy="0 0 0"/>
-            <mass value="30.0"/>
-            <inertia ixx="10.0" ixy="0.0" ixz="0.0" iyy="10.0" iyz="0.0" izz="10.0"/>
+            <origin xyz="0 0 0.1111" rpy="0 0 0"/>
+            <mass value="55.0"/>
+            <inertia ixx="1.700489" ixy="0.0" ixz="0.0" iyy="1.700489" iyz="0.0" izz="2.604803"/>
         </inertial>
     </link>
@@ -27,9 +27,9 @@
     </joint>
     <link name="front_hokuyo_link">
-        <inertial>
+        <!-- <inertial>
             <origin xyz="0 0 0" rpy="0 0 0"/>
             <mass value="1.0"/>
             <inertia ixx="1.0" ixy="0.0" ixz="0.0" iyy="1.0" iyz="0.0" izz="1.0"/>
-        </inertial>
+        </inertial> -->
     </link>
     <xacro:insert_hokuyo_sensor name="front" />
@@ -40,9 +40,9 @@
     </joint>
     <link name="rear_hokuyo_link">
-        <inertial>
+        <!-- <inertial>
             <origin xyz="0 0 0" rpy="0 0 0"/>
             <mass value="1.0"/>
             <inertia ixx="1.0" ixy="0.0" ixz="0.0" iyy="1.0" iyz="0.0" izz="1.0"/>
-        </inertial>
+        </inertial> -->
     </link>
     <xacro:insert_hokuyo_sensor name="rear" />
@@ -62,11 +62,11 @@
             <origin xyz="0 0 0" rpy="0 0 0"/>
             <geometry>
-                <mesh filename="package://living_lab_robot_description/meshes/omni_wheel.dae" scale="1 1 1"/>
+                <sphere radius="0.065"/>
             </geometry>
         </collision>
         <inertial>
-            <origin xyz="0 0 0" rpy="0 0 0"/>
-            <mass value="1.0"/>
-            <inertia ixx="1.0" ixy="0.0" ixz="0.0" iyy="1.0" iyz="0.0" izz="1.0"/>
+            <origin xyz="0 -0.0015 0" rpy="0 0 0"/>
+            <mass value="0.42"/>
+            <inertia ixx="0.000562" ixy="0.0" ixz="0.0" iyy="0.000884" iyz="0.0" izz="0.000562"/>
         </inertial>
     </link>
@@ -88,11 +88,11 @@
             <origin xyz="0 0 0" rpy="0 0 0"/>
             <geometry>
-                <mesh filename="package://living_lab_robot_description/meshes/omni_wheel.dae" scale="1 1 1"/>
+                <sphere radius="0.065"/>
             </geometry>
         </collision>
         <inertial>
-            <origin xyz="0 0 0" rpy="0 0 0"/>
-            <mass value="1.0"/>
-            <inertia ixx="1.0" ixy="0.0" ixz="0.0" iyy="1.0" iyz="0.0" izz="1.0"/>
+            <origin xyz="0 -0.0015 0" rpy="0 0 0"/>
+            <mass value="0.42"/>
+            <inertia ixx="0.000562" ixy="0.0" ixz="0.0" iyy="0.000884" iyz="0.0" izz="0.000562"/>
         </inertial>
     </link>
@@ -114,11 +114,11 @@
             <origin xyz="0 0 0" rpy="0 0 0"/>
             <geometry>
-                <mesh filename="package://living_lab_robot_description/meshes/omni_wheel.dae" scale="1 1 1"/>
+                <sphere radius="0.065"/>
             </geometry>
         </collision>
         <inertial>
-            <origin xyz="0 0 0" rpy="0 0 0"/>
-            <mass value="1.0"/>
-            <inertia ixx="1.0" ixy="0.0" ixz="0.0" iyy="1.0" iyz="0.0" izz="1.0"/>
+            <origin xyz="0 -0.0015 0" rpy="0 0 0"/>
+            <mass value="0.42"/>
+            <inertia ixx="0.000562" ixy="0.0" ixz="0.0" iyy="0.000884" iyz="0.0" izz="0.000562"/>
         </inertial>
     </link>
